Commit message: added first gazebo files, modified two_wheel_robot model

File: src/my_two_wheel_robot/urdf/my_two_wheel_robot.urdf.xacro (robot description, xacro)
@@ -1,172 +1,519 @@
 <?xml version="1.0"?>
 <robot name="visual">
-	<material name="blue">
-		<color rgba="0 0 1 1"/>
-	</material>
-	<material name="black">
-		<color rgba="0 0 0 1"/>
-	</material>
-	<material name="white">
-		<color rgba="1 1 1 1"/>
-	</material>
-	<!-- Odom link (корень без инерции) -->
-	<link name="odom"/>
-	<!-- Основная платформа (с инерцией) -->
-	<link name="base_link">
-		<visual>
-			<geometry>
-				<box size="0.2 0.23 0.005"/>
-			</geometry>
-			<material name="black"/>
-		</visual>
-		<collision>
-			<geometry>
-				<box size="0.2 0.23 0.005"/>
-			</geometry>
-		</collision>
-		<inertial>
-			<mass value="10"/>
-			<inertia ixx="1e-3" ixy="0" ixz="0"
-			         iyy="1e-3" iyz="0" izz="1e-3"/>
-		</inertial>
-	</link>
-	<joint name="base_link_joint" type="fixed">
-		<parent link="odom"/>
-		<child link="base_link"/>
-		<origin xyz="0 0 0" rpy="0 0 0"/>
-	</joint>
-	<!-- Промежуточное звено (left_base) -->
-	<link name="left_base">
-		<visual>
-			<geometry>
-				<box size="0.01 0.01 0.01"/>
-			</geometry>
-		</visual>
-	</link>
-	<joint name="left_base_joint" type="fixed">
-		<parent link="base_link"/>
-		<child link="left_base"/>
-		<!-- Joint находится в позиции оси колеса -->
-		<origin xyz="0.05 0.13 0"/>
-	</joint>
-	<!-- Левое колесо -->
-	<link name="left_wheel">
-		<visual>
-			<origin rpy="1.57075 0 0" xyz="0 0 0"/>
-			<geometry>
-				<cylinder length="0.025" radius="0.0325"/>
-			</geometry>
-			<material name="blue"/>
-		</visual>
-		<collision>
-			<origin rpy="1.57075 0 0" xyz="0 0 0"/>
-			<geometry>
-				<cylinder length="0.025" radius="0.0325"/>
-			</geometry>
-		</collision>
-		<inertial>
-			<mass value="1"/>
-			<inertia ixx="1e-3" ixy="0" ixz="0"
-			         iyy="1e-3" iyz="0" izz="1e-3"/>
-		</inertial>
-	</link>
-	<joint name="left_wheel_joint" type="continuous">
-		<axis xyz="0 1 0"/>
-		<parent link="left_base"/>
-		<child link="left_wheel"/>
-		<!-- Колесо на нулевой позиции относительно промежуточного звена -->
-		<origin xyz="0 0 0" rpy="0 0 0"/>
-		<command_interface name="velocity"/><!-- управляем скорость колеса -->
-		<state_interface name="position"/><!-- состояние: пройденный угол -->
-		<state_interface name="velocity"/><!-- состояние: текущая скорость -->
-	</joint>
-	<!-- Промежуточное звено (right_base) -->
-	<link name="right_base">
-		<visual>
-			<geometry>
-				<box size="0.01 0.01 0.01"/>
-			</geometry>
-		</visual>
-	</link>
-	<joint name="right_base_joint" type="fixed">
-		<parent link="base_link"/>
-		<child link="right_base"/>
-		<!-- Joint находится в позиции оси колеса -->
-		<origin xyz="0.05 -0.13 0"/>
-	</joint>
-	<!-- Правое колесо -->
-	<link name="right_wheel">
-		<visual>
-			<origin rpy="1.57075 0 0" xyz="0 0 0"/>
-			<geometry>
-				<cylinder length="0.025" radius="0.0325"/>
-			</geometry>
-			<material name="blue"/>
-		</visual>
-		<collision>
-			<origin rpy="1.57075 0 0" xyz="0 0 0"/>
-			<geometry>
-				<cylinder length="0.025" radius="0.0325"/>
-			</geometry>
-		</collision>
-		<inertial>
-			<mass value="1"/>
-			<inertia ixx="1e-3" ixy="0" ixz="0"
-			         iyy="1e-3" iyz="0" izz="1e-3"/>
-		</inertial>
-	</link>
-	<joint name="right_wheel_joint" type="continuous">
-		<axis xyz="0 1 0"/>
-		<parent link="right_base"/>
-		<child link="right_wheel"/>
-		<!-- Колесо на нулевой позиции относительно промежуточного звена -->
-		<origin xyz="0 0 0" rpy="0 0 0"/>
-		<command_interface name="velocity"/><!-- управляем скорость колеса -->
-		<state_interface name="position"/><!-- состояние: пройденный угол -->
-		<state_interface name="velocity"/><!-- состояние: текущая скорость -->
-	</joint>
-	<link name="caster_wheel">
-		<visual>
-			<origin xyz="0 0 0" rpy="0 0 0"/>
-			<geometry>
-				<sphere radius="0.015"/>
-			</geometry>
-			<material name="white"/>
-		</visual>
-		<collision>
-			<origin xyz="0 0 0" rpy="0 0 0"/>
-			<geometry>
-				<sphere radius="0.015"/>
-			</geometry>
-		</collision>
-		<inertial>
-			<mass value="0.1"/>
-			<inertia ixx="1e-4" ixy="0" ixz="0"
-			         iyy="1e-3" iyz="0" izz="1e-3"/>
-		</inertial>
-	</link>
-	<joint name="caster_wheel_joint" type="fixed">
-		<parent link="base_link"/>
-		<child link="caster_wheel"/>
-		<origin xyz="-0.09 0 -0.01"/>
-	</joint>
-	<ros2_control name="my_robot_hardware" type="system">
-		<hardware>
-			<!-- Подключаем эмуляцию аппаратной части: GenericSystem с вычислением динамики -->
-			<plugin>mock_components/GenericSystem</plugin>
-			<param name="update_rate" type="int">50</param>
-			<param name="calculate_dynamics" type="bool">true</param>
-		</hardware>
-		<!-- Описание управляемых шарниров -->
-		<joint name="left_wheel_joint">
-			<command_interface name="velocity"/><!-- управляем скорость колеса -->
-			<state_interface name="position"/><!-- состояние: пройденный угол -->
-			<state_interface name="velocity"/><!-- состояние: текущая скорость -->
-		</joint>
-		<joint name="right_wheel_joint">
-			<command_interface name="velocity"/>
-			<state_interface name="position"/>
-			<state_interface name="velocity"/>
-		</joint>
-	</ros2_control>
+  <!-- Определения материалов -->
+  <material name="blue">
+    <color rgba="0 0 1 1"/>
+  </material>
+  <material name="black">
+    <color rgba="0 0 0 1"/>
+  </material>
+  <material name="white">
+    <color rgba="1 1 1 1"/>
+  </material>
+  <material name="green">
+    <color rgba="0 0.7 0 1"/>
+  </material>
+  <!-- Корневое звено -->
+  <link name="odom"/>
+  <!-- ========== Первый уровень: основная платформа ========== -->
+  <link name="base_link">
+    <visual>
+      <geometry>
+        <box size="0.2 0.23 0.005"/>
+      </geometry>
+      <material name="black"/>
+    </visual>
+    <collision>
+      <geometry>
+        <box size="0.2 0.23 0.005"/>
+      </geometry>
+    </collision>
+    <inertial>
+      <mass value="1.5"/>
+      <inertia ixx="1e-3" ixy="0" ixz="0"
+               iyy="1e-3" iyz="0" izz="1e-3"/>
+    </inertial>
+  </link>
+  <joint name="base_link_joint" type="fixed">
+    <parent link="odom"/>
+    <child link="base_link"/>
+    <origin xyz="0 0 0" rpy="0 0 0"/>
+  </joint>
+    <!-- Материал для стоек (пример: серебристый) -->
+  <material name="silver">
+    <color rgba="0.8 0.8 0.8 1.0"/>
+  </material>
+  <!-- Четыре стойки (палки) от base_link к верхней платформе
+       Диаметр 10 мм => радиус 0.005 м
+       Длина ~0.19 м (от z=0.005 до z=0.195)
+       Располагаем их в углах (x=±0.09, y=±0.105) -->
+  <!-- Левая передняя стойка -->
+  <link name="rod_front_left">
+    <visual>
+      <!-- Поднимаем её центр на середину (0.095), смещаем в угол (x=+0.09, y=+0.105) -->
+      <origin xyz="0.09 0.105 0.095" rpy="0 0 0"/>
+      <geometry>
+        <cylinder length="0.19" radius="0.005"/>
+      </geometry>
+      <material name="silver"/>
+    </visual>
+    <collision>
+      <origin xyz="0.09 0.105 0.095" rpy="0 0 0"/>
+      <geometry>
+        <cylinder length="0.19" radius="0.005"/>
+      </geometry>
+    </collision>
+    <inertial>
+      <mass value="0.05"/>
+      <origin xyz="0.09 0.105 0.095" rpy="0 0 0"/>
+      <inertia ixx="1e-5" ixy="0" ixz="0"
+               iyy="1e-5" iyz="0" izz="1e-5"/>
+    </inertial>
+  </link>
+  <joint name="rod_front_left_joint" type="fixed">
+    <parent link="base_link"/>
+    <child link="rod_front_left"/>
+    <origin xyz="0 0 0" rpy="0 0 0"/>
+  </joint>
+  <!-- Правая передняя стойка -->
+  <link name="rod_front_right">
+    <visual>
+      <origin xyz="0.09 -0.105 0.095" rpy="0 0 0"/>
+      <geometry>
+        <cylinder length="0.19" radius="0.005"/>
+      </geometry>
+      <material name="silver"/>
+    </visual>
+    <collision>
+      <origin xyz="0.09 -0.105 0.095" rpy="0 0 0"/>
+      <geometry>
+        <cylinder length="0.19" radius="0.005"/>
+      </geometry>
+    </collision>
+    <inertial>
+      <mass value="0.05"/>
+      <origin xyz="0.09 -0.105 0.095" rpy="0 0 0"/>
+      <inertia ixx="1e-5" ixy="0" ixz="0"
+               iyy="1e-5" iyz="0" izz="1e-5"/>
+    </inertial>
+  </link>
+  <joint name="rod_front_right_joint" type="fixed">
+    <parent link="base_link"/>
+    <child link="rod_front_right"/>
+    <origin xyz="0 0 0" rpy="0 0 0"/>
+  </joint>
+  <!-- Левая задняя стойка -->
+  <link name="rod_rear_left">
+    <visual>
+      <origin xyz="-0.09 0.105 0.095" rpy="0 0 0"/>
+      <geometry>
+        <cylinder length="0.19" radius="0.005"/>
+      </geometry>
+      <material name="silver"/>
+    </visual>
+    <collision>
+      <origin xyz="-0.09 0.105 0.095" rpy="0 0 0"/>
+      <geometry>
+        <cylinder length="0.19" radius="0.005"/>
+      </geometry>
+    </collision>
+    <inertial>
+      <mass value="0.05"/>
+      <origin xyz="-0.09 0.105 0.095" rpy="0 0 0"/>
+      <inertia ixx="1e-5" ixy="0" ixz="0"
+               iyy="1e-5" iyz="0" izz="1e-5"/>
+    </inertial>
+  </link>
+  <joint name="rod_rear_left_joint" type="fixed">
+    <parent link="base_link"/>
+    <child link="rod_rear_left"/>
+    <origin xyz="0 0 0" rpy="0 0 0"/>
+  </joint>
+  <!-- Правая задняя стойка -->
+  <link name="rod_rear_right">
+    <visual>
+      <origin xyz="-0.09 -0.105 0.095" rpy="0 0 0"/>
+      <geometry>
+        <cylinder length="0.19" radius="0.005"/>
+      </geometry>
+      <material name="silver"/>
+    </visual>
+    <collision>
+      <origin xyz="-0.09 -0.105 0.095" rpy="0 0 0"/>
+      <geometry>
+        <cylinder length="0.19" radius="0.005"/>
+      </geometry>
+    </collision>
+    <inertial>
+      <mass value="0.05"/>
+      <origin xyz="-0.09 -0.105 0.095" rpy="0 0 0"/>
+      <inertia ixx="1e-5" ixy="0" ixz="0"
+               iyy="1e-5" iyz="0" izz="1e-5"/>
+    </inertial>
+  </link>
+  <joint name="rod_rear_right_joint" type="fixed">
+    <parent link="base_link"/>
+    <child link="rod_rear_right"/>
+    <origin xyz="0 0 0" rpy="0 0 0"/>
+  </joint>
+  <!-- Колёсная база (левая сторона) -->
+  <link name="left_base">
+    <visual>
+      <geometry>
+        <box size="0.01 0.01 0.01"/>
+      </geometry>
+    </visual>
+  </link>
+  <joint name="left_base_joint" type="fixed">
+    <parent link="base_link"/>
+    <child link="left_base"/>
+    <origin xyz="0.05 0.13 0" rpy="0 0 0"/>
+  </joint>
+  <link name="left_wheel">
+    <visual>
+      <origin rpy="1.57075 0 0" xyz="0 0 0"/>
+      <geometry>
+        <cylinder length="0.025" radius="0.0325"/>
+      </geometry>
+      <material name="blue"/>
+    </visual>
+    <collision>
+      <origin rpy="1.57075 0 0" xyz="0 0 0"/>
+      <geometry>
+        <cylinder length="0.025" radius="0.0325"/>
+      </geometry>
+    </collision>
+    <inertial>
+      <mass value="1"/>
+      <inertia ixx="1e-3" ixy="0" ixz="0"
+               iyy="1e-3" iyz="0" izz="1e-3"/>
+    </inertial>
+  </link>
+  <joint name="left_wheel_joint" type="continuous">
+    <axis xyz="0 1 0"/>
+    <parent link="left_base"/>
+    <child link="left_wheel"/>
+    <origin xyz="0 0 0" rpy="0 0 0"/>
+    <command_interface name="velocity"/>
+    <state_interface name="position"/>
+    <state_interface name="velocity"/>
+  </joint>
+  <!-- Колёсная база (правая сторона) -->
+  <link name="right_base">
+    <visual>
+      <geometry>
+        <box size="0.01 0.01 0.01"/>
+      </geometry>
+    </visual>
+  </link>
+  <joint name="right_base_joint" type="fixed">
+    <parent link="base_link"/>
+    <child link="right_base"/>
+    <origin xyz="0.05 -0.13 0" rpy="0 0 0"/>
+  </joint>
+  <link name="right_wheel">
+    <visual>
+      <origin rpy="1.57075 0 0" xyz="0 0 0"/>
+      <geometry>
+        <cylinder length="0.025" radius="0.0325"/>
+      </geometry>
+      <material name="blue"/>
+    </visual>
+    <collision>
+      <origin rpy="1.57075 0 0" xyz="0 0 0"/>
+      <geometry>
+        <cylinder length="0.025" radius="0.0325"/>
+      </geometry>
+    </collision>
+    <inertial>
+      <mass value="1"/>
+      <inertia ixx="1e-3" ixy="0" ixz="0"
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
Commit message: added launch file for easier gz-ros2 starting

File: src/my_two_wheel_robot/urdf/my_two_wheel_robot.urdf.xacro (robot description, xacro)
@@ -322,154 +322,4 @@
     <origin xyz="0 0 0.130" rpy="0 0 0"/>
   </joint>
-  <!-- ========== Манипулятор (установлен на верхней платформе) ========== -->
-  <!-- Сустав плеча: сдвигаем манипулятор вперёд на 0.05 м -->
-  <joint name="arm_shoulder_joint" type="revolute">
-    <parent link="top_plate"/>
-    <child link="arm_link1"/>
-    <origin xyz="0.1 0 0" rpy="0 0 0"/>
-    <!-- Используем ось вращения по Y для движения в плоскости (наклон вниз/вверх) -->
-    <axis xyz="0 1 0"/>
-    <limit lower="-1.57" upper="1.57" effort="5.0" velocity="1.0"/>
-  </joint>
-  <!-- Первое звено манипулятора (плечо), направлено вниз -->
-  <link name="arm_link1">
-    <visual>
-      <!-- Сдвиг на -0.04 по Z: центр звена ниже сочленения;
-           поворот на 180° по X (3.1416 рад) переворачивает звено -->
-      <origin xyz="0 0 -0.04" rpy="3.1416 0 0"/>
-      <geometry>
-        <cylinder length="0.08" radius="0.01"/>
-      </geometry>
-      <material name="green"/>
-    </visual>
-    <collision>
-      <origin xyz="0 0 -0.04" rpy="3.1416 0 0"/>
-      <geometry>
-        <cylinder length="0.08" radius="0.01"/>
-      </geometry>
-    </collision>
-    <inertial>
-      <mass value="0.2"/>
-      <origin xyz="0 0 -0.04" rpy="3.1416 0 0"/>
-      <inertia ixx="1e-3" ixy="0" ixz="0"
-               iyy="1e-3" iyz="0" izz="1e-3"/>
-    </inertial>
-  </link>
-  <!-- Сустав локтя: теперь расположен в конце первого звена -->
-  <joint name="arm_elbow_joint" type="revolute">
-    <parent link="arm_link1"/>
-    <child link="arm_link2"/>
-    <origin xyz="0 0 -0.08" rpy="0 0 0"/>
-    <axis xyz="0 1 0"/>
-    <limit lower="0" upper="2.8" effort="5.0" velocity="1.0"/>
-  </joint>
-  <!-- Второе звено манипулятора (локоть), также направлено вниз -->
-  <link name="arm_link2">
-    <visual>
-      <origin xyz="0 0 -0.04" rpy="3.1416 0 0"/>
-      <geometry>
-        <cylinder length="0.08" radius="0.01"/>
-      </geometry>
-      <material name="green"/>
-    </visual>
-    <collision>
-      <origin xyz="0 0 -0.04" rpy="3.1416 0 0"/>
-      <geometry>
-        <cylinder length="0.08" radius="0.01"/>
-      </geometry>
-    </collision>
-    <inertial>
-      <mass value="0.2"/>
-      <origin xyz="0 0 -0.04" rpy="3.1416 0 0"/>
-      <inertia ixx="1e-3" ixy="0" ixz="0"
-               iyy="1e-3" iyz="0" izz="1e-3"/>
-    </inertial>
-  </link>
-  <!-- Фиксированный сустав для крепления гриппера -->
-  <joint name="wrist_joint" type="fixed">
-    <parent link="arm_link2"/>
-    <child link="gripper_base"/>
-    <origin xyz="0 0 -0.08" rpy="0 0 0"/>
-  </joint>
-  <!-- Гриппер (база захвата) -->
-<link name="gripper_base">
-  <visual>
-    <origin xyz="0 0 0" rpy="0 0 0"/>
-    <geometry>
-      <sphere radius="0.02"/>
-    </geometry>
-    <material name="blue"/>
-  </visual>
-  <collision>
-    <origin xyz="0 0 0" rpy="0 0 0"/>
-    <geometry>
-      <sphere radius="0.01"/>
-    </geometry>
-  </collision>
-  <inertial>
-    <mass value="0.1"/>
-    <origin xyz="0 0 0" rpy="0 0 0"/>
-    <inertia ixx="1e-4" ixy="0" ixz="0"
-             iyy="1e-4" iyz="0" izz="1e-4"/>
-  </inertial>
-</link>
-<!-- Левый палец -->
-<link name="finger_left">
-  <visual>
-    <origin xyz="0 0.025 -0.015" rpy="0 0 90"/>
-    <geometry>
-      <cylinder length="0.05" radius="0.005"/>
-    </geometry>
-    <material name="blue"/>
-  </visual>
-  <collision>
-    <origin xyz="0 0.025 -0.015" rpy="0 0 90"/>
-    <geometry>
-      <cylinder length="0.05" radius="0.005"/>
-    </geometry>
-  </collision>
-  <inertial>
-    <mass value="0.01"/>
-    <origin xyz="0 0.025 -0.015" rpy="0 0 90"/>
-    <inertia ixx="1e-4" ixy="0" ixz="0"
-             iyy="1e-4" iyz="0" izz="1e-4"/>
-  </inertial>
-</link>
-<joint name="finger_left_joint" type="revolute">
-  <parent link="gripper_base"/>
-  <child link="finger_left"/>
-  <origin xyz="0 0 -0.01" rpy="0 0 0"/>
-  <axis xyz="-1 0 0"/><!-- Исправлено направление вращения -->
-  <limit lower="0" upper="0.5" effort="2.0" velocity="1.0"/>
-</joint>
-<!-- Правый палец -->
-<link name="finger_right">
-  <visual>
-    <origin xyz="0 -0.025 -0.015" rpy="0 0 90"/>
-    <geometry>
-      <cylinder length="0.05" radius="0.005"/>
-    </geometry>
-    <material name="blue"/>
-  </visual>
-  <collision>
-    <origin xyz="0 -0.025 -0.015" rpy="0 0 90"/>
-    <geometry>
-      <cylinder length="0.05" radius="0.005"/>
-    </geometry>
-  </collision>
-  <inertial>
-    <mass value="0.01"/>
-    <origin xyz="0 -0.025 -0.015" rpy="0 0 90"/>
-    <inertia ixx="1e-4" ixy="0" ixz="0"
-             iyy="1e-4" iyz="0" izz="1e-4"/>
-  </inertial>
-</link>
-<joint name="finger_right_joint" type="revolute">
-  <parent link="gripper_base"/>
-  <child link="finger_right"/>
-  <origin xyz="0 0 -0.01" rpy="0 0 0"/>
-  <axis xyz="1 0 0"/>
-  <limit lower="0" upper="0.5" effort="2.0" velocity="1.0"/>
-</joint>
   <!-- ========== Лидар (на верхней платформе) ========== -->
   <link name="lidar_link">
