Commit message: fixed robot model, bridge, controllers etc. robot already moving in sim and rviz2, rviz2 showing current lidar scan

File: src/my_two_wheel_robot/urdf/dif_robot_description/dif_robot.urdf.xacro (robot description, xacro)
@@ -122,5 +122,5 @@
         <origin xyz="0 0 0" rpy="0 0 0"/>
         <geometry>
-            <sphere radius="0.015"/>
+            <sphere radius="0.01625"/>
         </geometry>
         <material name="white"/>
@@ -129,5 +129,5 @@
         <origin xyz="0 0 0" rpy="0 0 0"/>
         <geometry>
-            <sphere radius="0.015"/>
+            <sphere radius="0.01625"/>
         </geometry>
         </collision>
@@ -141,5 +141,5 @@
         <parent link="base_link"/>
         <child link="caster_wheel"/>
-        <origin xyz="-0.09 0 -0.015" rpy="0 0 0"/>
+        <origin xyz="-0.09 0 -0.01625" rpy="0 0 0"/>
     </joint>
     <!-- ========== Второй уровень: плата электроники ========== -->
@@ -225,36 +225,27 @@
         <origin xyz="0 0 0" rpy="0 0 0"/>
     </joint>
+    <!-- Gazebo sensor -->
     <gazebo reference="lidar_link">
-    <sensor name="lidar_sensor" type="gpu_ray">
-        <pose>0 0 0 0 0 0</pose>
+    <sensor name="gpu_lidar" type="gpu_lidar">
+        <update_rate>10</update_rate>
+        <topic>lidar_scan</topic>
+        <gz_frame_id>lidar_link</gz_frame_id>
+        <lidar>
+        <scan>
+            <horizontal>
+            <samples>720</samples>
+            <resolution>1</resolution>
+            <min_angle>-3.14159</min_angle>
+            <max_angle>3.14159</max_angle>
+            </horizontal>
+        </scan>
+        <range>
+            <min>0.05</min>
+            <max>10.0</max>
+            <resolution>0.01</resolution>
+        </range>
+        </lidar>
         <always_on>true</always_on>
         <visualize>true</visualize>
-        <update_rate>10</update_rate>
-        <ray>
-        <scan>
-            <horizontal>
-            <samples>36</samples>
-            <resolution>1</resolution>
-            <min_angle>-1.5708</min_angle>
-            <max_angle>1.5708</max_angle>
-            </horizontal>
-            <vertical>
-            <samples>1</samples>
-            <resolution>1</resolution>
-            <min_angle>0</min_angle>
-            <max_angle>0</max_angle>
-            </vertical>
-        </scan>
-        <range>
-            <min>0.08</min>
-            <max>2.0</max>
-            <resolution>0.01</resolution>
-        </range>
-        <noise>
-            <type>gaussian</type>
-            <mean>0.0</mean>
-            <stddev>0.01</stddev>
-        </noise>
-        </ray>
     </sensor>
     </gazebo>
@@ -262,7 +253,8 @@
     <ros2_control name="my_robot_hardware" type="system">
         <hardware>
-        <plugin>mock_components/GenericSystem</plugin>
+            <plugin>gz_ros2_control/GazeboSimSystem</plugin>
+        <!-- <plugin>mock_components/GenericSystem</plugin>
         <param name="update_rate" type="int">50</param>
-        <param name="calculate_dynamics" type="bool">true</param>
+        <param name="calculate_dynamics" type="bool">true</param> -->
         </hardware>
         <joint name="left_wheel_joint">
@@ -278,6 +270,5 @@
     </ros2_control>
     <gazebo>
-        <plugin name="gz_ros2_control"
-                filename="libgz_ros2_control-system.so">
+        <plugin name="gz_ros2_control::GazeboSimROS2ControlPlugin" filename="libgz_ros2_control-system.so">
             <!-- Имя модели в Gazebo (model name) должно совпадать с тем,
                 под которым ты спавнишь робота. Часто можно не указывать,
@@ -287,4 +278,7 @@
             <!-- Можно задать namespace, если нужно -->
             <!-- <robot_namespace>/my_robot</robot_namespace> -->
+            <!-- <parameters>$(find my_two_wheel_robot)/config/diff_drive_controllers.yaml</parameters> -->
+            <!-- new_dd_controllers.yaml -->
+            <parameters>/home/ager/ros2_ws/install/my_two_wheel_robot/share/my_two_wheel_robot/config/dd_controllers.yaml</parameters>
         </plugin>
     </gazebo>
